File: PowerSlice/PowerSlice.kicad_sch (KiCad schematic)
At the start: 35 parts, among them J1 Conn_01x10_Pin, J2 DC_In_Barrel, J3 DC_In_Screw, J4 ESTOP, J5 +12V_Screw, J6 +5V_Screw, J7 +3V3_Screw, U1 PTH08080WAD, U2 PTH08080WAD, U3 INA214BIDCKR, U4 INA214BIDCKR, U5 INA214BIDCKR, U6 NUCLEO-F303K8

Commit message: "Final" edits before submission for ordering
Parts:
- removed J5: +12V_Screw, 691137710002:691137710002, symbol Connector:Screw_Terminal_01x02
- removed J6: +5V_Screw, 691137710002:691137710002, symbol Connector:Screw_Terminal_01x02
- removed J7: +3V3_Screw, 691137710002:691137710002, symbol Connector:Screw_Terminal_01x02
- added TP1, TP10, TP11, TP12, TP13, TP14, TP2, TP3, TP4, TP5, TP6, TP7, TP8, TP9: TestPoint, TestPoint:TestPoint_Keystone_5005-5009_Compact, symbol Connector:TestPoint
- renumbered C3 to C1, C4 to C2, C1 to C3, C2 to C4, C7 to C5, C5 to C7, U5 to U3, U3 to U5
Connections:
- net +12V: now also TP1.1
- net +3V3: now also TP3.1
- net +5V: now also TP2.1
- net 12VSns: now also TP9.1
- net 3V3Sns: now also TP11.1
- net 5VSns: now also TP10.1
- net GND: now also TP12.1, TP4.1, TP8.1
- net R1_Current: now also TP5.1
- net R2_Current: now also TP6.1
- net R3_Current: now also TP7.1
- net SCL: now also TP14.1
- net SDA: now also TP13.1
Other:
- moved on the sheet: C5, C6, C7, F1, F2, F3, J1, R1, R10, R11, R2, R3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
